File: KiCad/PMod_ADDAC/IO.sch (KiCad schematic (older format))
At the start: 25 parts

Commit message: kicad update
Parts:
- removed R? (x2): R, symbol Device:R
- removed U? (x5): OPAMP, symbol pspice:OPAMP
- added C12: variable, Capacitor_THT:C_Disc_D5.0mm_W2.5mm_P5.00mm, symbol Device:C_Small
- added C? (x4): 10n, Capacitor_SMD:C_0805_2012Metric_Pad1.15x1.40mm_HandSolder, symbol Device:C_Small
- added R25, R26: 200, symbol Device:R
- added R27: 1k, symbol Device:R
- added RV1: 10k, symbol Device:R_POT_TRIM
- added RV2: 10k, Potentiometer_THT:Potentiometer_Bourns_3339P_Vertical, symbol Device:R_POT_TRIM
- added U1, U2, U3: TL072, symbol Amplifier_Operational:TL072
- C8: renamed from C?; footprint (none) -> Capacitor_SMD:C_0805_2012Metric_Pad1.15x1.40mm_HandSolder
- C9: renamed from C?; value C_Small -> variable; footprint (none) -> Capacitor_THT:C_Disc_D5.0mm_W2.5mm_P5.00mm
- R20: renamed from R?; footprint (none) -> Resistor_SMD:R_0805_2012Metric_Pad1.15x1.40mm_HandSolder
- gave numbers to parts that had none: 15
Connections:
- net labels added: +12V, -12V
- wire segments 61 -> 89
Other:
- note added: "Vout=-Vin/(j*omega*R*C)"
- note added: "multiple caps for different frequencies? summing amplifier to collect the different frequencies???"
- moved on the sheet: R31
