File: KiCad/PMod_ADDAC/R2R.sch (KiCad schematic (older format))
At the start: 24 parts

Commit message: kicad update
Parts:
- removed U? (x2): TSX632, Package_SO:SOIC-8_3.9x4.9mm_P1.27mm, symbol Device:Opamp_Dual_Generic
- added C?: 100, Capacitor_SMD:C_0805_2012Metric_Pad1.15x1.40mm_HandSolder, symbol Device:C_Small
- added U2, U?: TL072, symbol Amplifier_Operational:TL072
- gave numbers to parts that had none: 22
Connections:
- net GND: now also C?.1
- net VCC: no longer C1.1
- net at JP1.1 (A), R10.1, R9.2: now also U2.5 (+)
- net at JP1.2 (B), R19.1: now also U2.6 (-), U2.7
- new net +12V: C?.2, U?.8 (V+)
- new net -12V: C1.1, U?.4 (V-)
