File: KiCad/PMod_ADDAC/power.sch (KiCad schematic (older format))
At the start: 10 parts

Commit message: kicad update
Parts:
- added J2: Basys power, Connector_PinHeader_2.54mm:PinHeader_1x02_P2.54mm_Vertical, symbol Connector:Conn_01x02_Male
- gave numbers to parts that had none: 10
Connections:
- net +5V: now also J2.1 (Pin_1)
- net GND: now also J2.2 (Pin_2)
Changed lines of the file:
@@
 $Descr A4 11693 8268
 encoding utf-8
-Sheet 5 5
+Sheet 3 4
 Title ""
 Date ""
@@
 P 9650 4850
 AR Path="/62454E97" Ref="J?"  Part="1"
-AR Path="/6244F096/62454E97" Ref="J?"  Part="1"
-F 0 "J?" H 9622 4824 50  0000 R CNN
+AR Path="/6244F096/62454E97" Ref="J3"  Part="1"
+F 0 "J3" H 9622 4824 50  0000 R CNN
 F 1 "Conn_01x16_Male" H 9622 4733 50  0000 R CNN
 F 2 "Connector_PinHeader_2.54mm:PinHeader_2x08_P2.54mm_Vertical" H 9650 4850 50  0001 C CNN
@@
 P 8850 4250
 AR Path="/62454EAB" Ref="C?"  Part="1"
-AR Path="/6244F096/62454EAB" Ref="C?"  Part="1"
-F 0 "C?" H 8942 4296 50  0000 L CNN
+AR Path="/6244F096/62454EAB" Ref="C5"  Part="1"
+F 0 "C5" H 8942 4296 50  0000 L CNN
 F 1 "10n" H 8942 4205 50  0000 L CNN
 F 2 "" H 8850 4250 50  0001 C CNN
@@
 P 8850 4950
 AR Path="/62454EB1" Ref="C?"  Part="1"
-AR Path="/6244F096/62454EB1" Ref="C?"  Part="1"
-F 0 "C?" H 8942 4996 50  0000 L CNN
+AR Path="/6244F096/62454EB1" Ref="C6"  Part="1"
+F 0 "C6" H 8942 4996 50  0000 L CNN
 F 1 "10n" H 8942 4905 50  0000 L CNN
 F 2 "" H 8850 4950 50  0001 C CNN
@@
 P 8550 4950
 AR Path="/62454EB7" Ref="C?"  Part="1"
-AR Path="/6244F096/62454EB7" Ref="C?"  Part="1"
-F 0 "C?" H 8462 4904 50  0000 R CNN
+AR Path="/6244F096/62454EB7" Ref="C3"  Part="1"
+F 0 "C3" H 8462 4904 50  0000 R CNN
 F 1 "47u" H 8462 4995 50  0000 R CNN
 F 2 "" H 8550 4950 50  0001 C CNN
@@
 P 8550 4250
 AR Path="/62454EBD" Ref="C?"  Part="1"
-AR Path="/6244F096/62454EBD" Ref="C?"  Part="1"
-F 0 "C?" H 8462 4204 50  0000 R CNN
+AR Path="/6244F096/62454EBD" Ref="C2"  Part="1"
+F 0 "C2" H 8462 4204 50  0000 R CNN
 F 1 "47u" H 8462 4295 50  0000 R CNN
 F 2 "" H 8550 4250 50  0001 C CNN
@@
 P 9200 4150
 AR Path="/62454EC3" Ref="FB?"  Part="1"
-AR Path="/6244F096/62454EC3" Ref="FB?"  Part="1"
-F 0 "FB?" V 9055 4150 50  0000 C CNN
+AR Path="/6244F096/62454EC3" Ref="FB1"  Part="1"
+F 0 "FB1" V 9055 4150 50  0000 C CNN
 F 1 "Ferrite_Bead_Small" V 9054 4150 50  0001 C CNN
 F 2 "" V 9130 4150 50  0001 C CNN
@@
 P 9250 5050
 AR Path="/62454ECE" Ref="FB?"  Part="1"
-AR Path="/6244F096/62454ECE" Ref="FB?"  Part="1"
-F 0 "FB?" V 9105 5050 50  0000 C CNN
+AR Path="/6244F096/62454ECE" Ref="FB2"  Part="1"
+F 0 "FB2" V 9105 5050 50  0000 C CNN
 F 1 "Ferrite_Bead_Small" V 9104 5050 50  0001 C CNN
 F 2 "" V 9180 5050 50  0001 C CNN
@@
 P 9450 4600
 AR Path="/62454EE0" Ref="#PWR?"  Part="1"
-AR Path="/6244F096/62454EE0" Ref="#PWR?"  Part="1"
-F 0 "#PWR?" H 9450 4350 50  0001 C CNN
+AR Path="/6244F096/62454EE0" Ref="#PWR012"  Part="1"
+F 0 "#PWR012" H 9450 4350 50  0001 C CNN
 F 1 "GND" V 9455 4472 50  0000 R CNN
 F 2 "" H 9450 4600 50  0001 C CNN
@@
 P 8550 5050
 AR Path="/62454EE8" Ref="#PWR?"  Part="1"
-AR Path="/6244F096/62454EE8" Ref="#PWR?"  Part="1"
-F 0 "#PWR?" H 8550 4900 50  0001 C CNN
+AR Path="/6244F096/62454EE8" Ref="#PWR06"  Part="1"
+F 0 "#PWR06" H 8550 4900 50  0001 C CNN
 F 1 "+12V" H 8565 5223 50  0000 C CNN
 F 2 "" H 8550 5050 50  0001 C CNN
@@
 P 8700 4150
 AR Path="/62454EEE" Ref="#PWR?"  Part="1"
-AR Path="/6244F096/62454EEE" Ref="#PWR?"  Part="1"
-F 0 "#PWR?" H 8700 4250 50  0001 C CNN
+AR Path="/6244F096/62454EEE" Ref="#PWR08"  Part="1"
+F 0 "#PWR08" H 8700 4250 50  0001 C CNN
 F 1 "-12V" H 8715 4323 50  0000 C CNN
 F 2 "" H 8700 4150 50  0001 C CNN
@@
 P 8850 5350
 AR Path="/62454EF6" Ref="C?"  Part="1"
-AR Path="/6244F096/62454EF6" Ref="C?"  Part="1"
-F 0 "C?" H 8942 5396 50  0000 L CNN
+AR Path="/6244F096/62454EF6" Ref="C7"  Part="1"
+F 0 "C7" H 8942 5396 50  0000 L CNN
 F 1 "10n" H 8942 5305 50  0000 L CNN
 F 2 "" H 8850 5350 50  0001 C CNN
@@
 P 8550 5350
 AR Path="/62454EFC" Ref="C?"  Part="1"
-AR Path="/6244F096/62454EFC" Ref="C?"  Part="1"
-F 0 "C?" H 8462 5304 50  0000 R CNN
+AR Path="/6244F096/62454EFC" Ref="C4"  Part="1"
+F 0 "C4" H 8462 5304 50  0000 R CNN
 F 1 "47u" H 8462 5395 50  0000 R CNN
 F 2 "" H 8550 5350 50  0001 C CNN
@@
 P 9250 5250
 AR Path="/62454F02" Ref="FB?"  Part="1"
-AR Path="/6244F096/62454F02" Ref="FB?"  Part="1"
-F 0 "FB?" V 9105 5250 50  0000 C CNN
+AR Path="/6244F096/62454F02" Ref="FB3"  Part="1"
+F 0 "FB3" V 9105 5250 50  0000 C CNN
 F 1 "Ferrite_Bead_Small" V 9104 5250 50  0001 C CNN
 F 2 "" V 9180 5250 50  0001 C CNN
@@
 P 8700 5450
 AR Path="/62454F0E" Ref="#PWR?"  Part="1"
-AR Path="/6244F096/62454F0E" Ref="#PWR?"  Part="1"
-F 0 "#PWR?" H 8700 5200 50  0001 C CNN
+AR Path="/6244F096/62454F0E" Ref="#PWR09"  Part="1"
+F 0 "#PWR09" H 8700 5200 50  0001 C CNN
 F 1 "GND" H 8705 5277 50  0000 C CNN
 F 2 "" H 8700 5450 50  0001 C CNN
@@
 P 8550 5250
 AR Path="/62454F18" Ref="#PWR?"  Part="1"
-AR Path="/6244F096/62454F18" Ref="#PWR?"  Part="1"
-F 0 "#PWR?" H 8550 5100 50  0001 C CNN
+AR Path="/6244F096/62454F18" Ref="#PWR07"  Part="1"
+F 0 "#PWR07" H 8550 5100 50  0001 C CNN
 F 1 "+5V" V 8565 5378 50  0000 L CNN
 F 2 "" H 8550 5250 50  0001 C CNN
@@
 $EndComp
 Connection ~ 8550 5250
+$Comp
+L Connector:Conn_01x02_Male J2
+U 1 1 6245A5F5
+P 8650 3350
+F 0 "J2" H 8758 3531 50  0000 C CNN
+F 1 "Basys power" H 8758 3440 50  0000 C CNN
+F 2 "Connector_PinHeader_2.54mm:PinHeader_1x02_P2.54mm_Vertical" H 8650 3350 50  0001 C CNN
+F 3 "~" H 8650 3350 50  0001 C CNN
+	1    8650 3350
+	1    0    0    -1
+$EndComp
+$Comp
+L power:+5V #PWR?
+U 1 1 6245B65C
+P 9000 3350
+AR Path="/6245B65C" Ref="#PWR?"  Part="1"
+AR Path="/6244F096/6245B65C" Ref="#PWR010"  Part="1"
+F 0 "#PWR010" H 9000 3200 50  0001 C CNN
+F 1 "+5V" V 9015 3478 50  0000 L CNN
+F 2 "" H 9000 3350 50  0001 C CNN
+F 3 "" H 9000 3350 50  0001 C CNN
+	1    9000 3350
+	0    1    1    0
+$EndComp
+Wire Wire Line
+	9000 3350 8850 3350
+$Comp
+L power:GND #PWR011
+U 1 1 6245BE5D
+P 9000 3450
+F 0 "#PWR011" H 9000 3200 50  0001 C CNN
+F 1 "GND" V 9005 3322 50  0000 R CNN
+F 2 "" H 9000 3450 50  0001 C CNN
+F 3 "" H 9000 3450 50  0001 C CNN
+	1    9000 3450
+	0    -1   -1   0
+$EndComp
+Wire Wire Line
+	9000 3450 8850 3450
 $EndSCHEMATC
