File: ADDAC/KiCad/PMod_ADDAC/_autosave-IO.sch (KiCad schematic (older format))
At the start: 45 parts, among them J4 AudioJack2_SwitchT, J5 AudioJack2_SwitchT, J6 Conn_01x03_Male, U1 TL072, U2 TL072, U3 TL072, U4 LM339

Commit message: Arduino tests
Other:
- note removed: "- diode skal tillade strøm fra R_logic igennem"
Changed lines of the file:
@@
 Wire Wire Line
 	9300 2250 9900 2250
-Text Notes 4800 5300 0    50   ~ 0
-- diode skal tillade strøm fra R_logic igennem
 $Comp
 L pspice:DIODE D1
