File: ADDAC/KiCad/PMod_ADDAC/power.sch (KiCad schematic (older format))
At the start: 11 parts, among them J2 Basys power, J3 Conn_01x16_Male

Commit message: PCB-progress
Parts:
- added JP2, JP3, JP4: Jumper_NO_Small, Resistor_THT:R_Axial_DIN0204_L3.6mm_D1.6mm_P1.90mm_Vertical, symbol Device:Jumper_NO_Small
- C2, C3, C4: footprint (none) -> Capacitor_THT:CP_Radial_D6.3mm_P2.50mm
- FB1, FB2, FB3: footprint (none) -> Resistor_SMD:R_0805_2012Metric_Pad1.15x1.40mm_HandSolder
- J3: value Conn_01x16_Male -> Eurorack Power Connector
Connections:
- net +12V: now also JP3.1
- net +5V: now also JP4.2
- net -12V: now also JP2.1
- net at FB1.1, J3.1 (Pin_1), J3.2 (Pin_2): now also JP2.2
- net at FB2.1, J3.10 (Pin_10), J3.9 (Pin_9): now also JP3.2
- net at FB3.1, J3.11 (Pin_11), J3.12 (Pin_12): now also JP4.1
Other:
- note added: "-12\nGnd\nGnd\nGnd\n+12\n+5\nCV\nGate"
- note removed: "-12\nGnd\n+12\n+5\nCV\nGate"
- moved on the sheet: C2, C3, C4, C5, C6, C7, FB1, FB2, FB3
