File: ADDAC/KiCad/PMod_ADDAC/IO.sch (KiCad schematic (older format))
At the start: 32 parts, among them J4 AudioJack2_SwitchT, J5 AudioJack2_SwitchT, U1 TL072, U2 TL072, U3 TL072

Commit message: PCB-progress
Parts:
- added C20, C21: 47n, Capacitor_SMD:C_0805_2012Metric_Pad1.15x1.40mm_HandSolder, symbol Device:C_Small
- added C22, C23, C27, C28, C29, C30: 100n, Capacitor_SMD:C_0805_2012Metric_Pad1.15x1.40mm_HandSolder, symbol Device:C_Small
- added C24, C31: 15p, Capacitor_SMD:C_0805_2012Metric_Pad1.15x1.40mm_HandSolder, symbol Device:C_Small
- added C25, C26: 10n, Capacitor_SMD:C_0805_2012Metric_Pad1.15x1.40mm_HandSolder, symbol Device:C_Small
- added J6: Conn_01x03_Male, Connector_PinHeader_2.54mm:PinHeader_1x03_P2.54mm_Vertical, symbol Connector:Conn_01x03_Male
- added R34: 4k, Resistor_SMD:R_0805_2012Metric_Pad1.15x1.40mm_HandSolder, symbol Device:R
- added R35: 1k, Resistor_SMD:R_0805_2012Metric_Pad1.15x1.40mm_HandSolder, symbol Device:R
- added R36: 200, Resistor_SMD:R_0805_2012Metric_Pad1.15x1.40mm_HandSolder, symbol Device:R
- added R37: 10k, Resistor_SMD:R_0805_2012Metric_Pad1.15x1.40mm_HandSolder, symbol Device:R
- added U4: LM339, Package_SO:SOIC-14_3.9x8.7mm_P1.27mm, symbol Comparator:LM339
- added U5: TL072, Package_SO:SOIC-8_3.9x4.9mm_P1.27mm, symbol Amplifier_Operational:TL072
- R26: value 200 -> 10k
- gave numbers to parts that had none: 1
Connections:
- net labels added: DAC_R2R_out
- wire segments 91 -> 141
Other:
- note added: "-high slew rate comparators (LMP7300MAX/NOPB)\n- TLV320\n- Lm339dr\n+-12 eller ?\ninput and outputs must be at 200 ohms, with at max 3.3V (?)\n"
- note added: "DAC"
- note removed: "- sends out voltage. High input impedance?"
- note removed: "-high slew rate comparators (LMP7300MAX/NOPB)\n+-12 eller ?\ninput and outputs must be at 200 ohms, with at max 3.3V (?)\n"

Commit message: Schematic
Parts:
- removed C26: 10n, Capacitor_SMD:C_0805_2012Metric_Pad1.15x1.40mm_HandSolder, symbol Device:C_Small
- removed C28: 100n, Capacitor_SMD:C_0805_2012Metric_Pad1.15x1.40mm_HandSolder, symbol Device:C_Small
- removed R30, R31, R35: 1k, Resistor_SMD:R_0805_2012Metric_Pad1.15x1.40mm_HandSolder, symbol Device:R
- removed R34: 4k, Resistor_SMD:R_0805_2012Metric_Pad1.15x1.40mm_HandSolder, symbol Device:R
Connections:
- net +12V: no longer C25.2, C27.2, U5.8 (V+)
- net +5V: now also C25.2, C27.2, U5.8 (V+)
- net -12V: no longer U5.4 (V-)
- net GND: now also U5.4 (V-); no longer U5.5 (+)
- net at C14.2, R32.2, U3.7: now also U3.6 (-)
- net at C24.1, R26.2, U4.2: now also U5.5 (+)
- net at R36.2: now also U5.6 (-), U5.7; no longer U5.1
- net at U5.2 (-): now also U5.1
Other:
- note added: "- high speed opamp eller anden løsning\n"
- note added: "DAC + output\n"
- note added: "diode + 0 til 5 v supply\n"
- note added: "input buffer + filter\n"
- note removed: "DAC"
- moved on the sheet: C25, C27, J6, R36, U4C, U4D, U5A, U5B

Commit message: PCB
Parts:
- removed C21: 47n, Capacitor_SMD:C_0805_2012Metric_Pad1.15x1.40mm_HandSolder, symbol Device:C_Small
- removed C23, C27: 100n, Capacitor_SMD:C_0805_2012Metric_Pad1.15x1.40mm_HandSolder, symbol Device:C_Small
- removed C25: 10n, Capacitor_SMD:C_0805_2012Metric_Pad1.15x1.40mm_HandSolder, symbol Device:C_Small
- removed U5: TL072, Package_SO:SOIC-8_3.9x4.9mm_P1.27mm, symbol Amplifier_Operational:TL072
- added D1: BAT43, Diode_THT:D_DO-35_SOD27_P7.62mm_Horizontal, symbol pspice:DIODE
- added D?: 3v9, Diode_THT:D_DO-41_SOD81_P10.16mm_Horizontal, symbol Device:D_Zener
- added R30, R?: 0, Resistor_THT:R_Axial_DIN0204_L3.6mm_D1.6mm_P1.90mm_Vertical, symbol Device:R
- added R?: 1k, Resistor_SMD:R_0805_2012Metric_Pad1.15x1.40mm_HandSolder, symbol Device:R
Connections:
- net +12V: no longer C20.2, C22.2, U4.3 (V+)
- net +5V: now also R30.2; no longer R26.1
- net -12V: no longer U4.12 (V-)
- net DAC_D_out: now also R?.2; no longer R27.2
- net GND: now also U4.12 (V-), D?.2 (A); no longer U4.10 (-), U4.13, U4.14, U4.8 (-)
- net at C24.1, R26.2, U4.2: now also D1.1 (K)
- net at R36.2: now also D1.2 (A)
- new net: D?.1 (K), R27.2, R?.1
- new net: C20.2, C22.2, R30.1, U4.3 (V+)
- new net: U4.10 (-), U4.13
- new net: U4.14, U4.8 (-)
- new net: R26.1, R?.2
- new net VCC: R?.1
Other:
- note added: "- diode skal tillade strøm fra R_logic igennem"
- note added: "- output current protection\n- diode...\n\n"
- note added: "- vcc fra board ind et eller andet sted?\n- jumper så man får power fra +-12V\n"
- note removed: "- high speed opamp eller anden løsning\n"
- note removed: "-high slew rate comparators (LMP7300MAX/NOPB)\n- TLV320\n- Lm339dr\n+-12 eller ?\ninput and outputs must be at 200 ohms, with at max 3.3V (?)\n"
- note removed: "diode + 0 til 5 v supply\n"
- moved on the sheet: R36, U4C

Commit message: pcb done?
Parts:
- gave numbers to parts that had none: 3
Changed lines of the file:
@@
 - vcc fra board ind et eller andet sted?\n- jumper så man får power fra +-12V\n
 $Comp
-L Device:R R?
+L Device:R R31
 U 1 1 6257E521
 P 4050 5300
-F 0 "R?" V 3843 5300 50  0000 C CNN
+F 0 "R31" V 3843 5300 50  0000 C CNN
 F 1 "0" V 3934 5300 50  0000 C CNN
 F 2 "Resistor_THT:R_Axial_DIN0204_L3.6mm_D1.6mm_P1.90mm_Vertical" V 3980 5300 50  0001 C CNN
@@
 - output current protection\n- diode...\n\n
 $Comp
-L Device:D_Zener D?
+L Device:D_Zener D2
 U 1 1 625A9B81
 P 6350 1800
-F 0 "D?" V 6304 1879 50  0000 L CNN
+F 0 "D2" V 6304 1879 50  0000 L CNN
 F 1 "3v9" V 6395 1879 50  0000 L CNN
 F 2 "Diode_THT:D_DO-41_SOD81_P10.16mm_Horizontal" H 6350 1800 50  0001 C CNN
@@
 $EndComp
 $Comp
-L power:GND #PWR?
+L power:GND #PWR024
 U 1 1 625AA06C
 P 6350 1950
-F 0 "#PWR?" H 6350 1700 50  0001 C CNN
+F 0 "#PWR024" H 6350 1700 50  0001 C CNN
 F 1 "GND" H 6355 1777 50  0000 C CNN
 F 2 "" H 6350 1950 50  0001 C CNN
@@
 	6350 1650 6750 1650
 $Comp
-L Device:R R?
+L Device:R R34
 U 1 1 625B7193
 P 6200 1650
-F 0 "R?" V 5993 1650 50  0000 C CNN
+F 0 "R34" V 5993 1650 50  0000 C CNN
 F 1 "1k" V 6084 1650 50  0000 C CNN
 F 2 "Resistor_SMD:R_0805_2012Metric_Pad1.15x1.40mm_HandSolder" V 6130 1650 50  0001 C CNN
