File: ADDAC/KiCad/PMod_ADDAC/PMod_ADDAC.kicad_pcb (KiCad board)
At the start: 2 copper layers, 35.6 x 21.1 mm, 31 parts, among them J1 Conn_01x12_Male, J2 Basys power, J3 Conn_01x16_Male, J4 AudioJack2_SwitchT, J5 AudioJack2_SwitchT

Commit message: updated PCB
Parts:
- added C10: 10n, Capacitor_SMD:C_0805_2012Metric_Pad1.15x1.40mm_HandSolder, F.Cu at (50.8, 99.7)
- added C11: 10n, Capacitor_SMD:C_0805_2012Metric_Pad1.15x1.40mm_HandSolder, F.Cu at (50.8, 102.9)
- added C13: 10n, Capacitor_SMD:C_0805_2012Metric_Pad1.15x1.40mm_HandSolder, F.Cu at (70.1, 58.1)
- added C14: 10n, Capacitor_SMD:C_0805_2012Metric_Pad1.15x1.40mm_HandSolder, F.Cu at (87.8, 42.4)
- added C15: 100, Capacitor_SMD:C_0805_2012Metric_Pad1.15x1.40mm_HandSolder, F.Cu at (115.6, 42.4)
- added C16: 10n, Capacitor_SMD:C_0805_2012Metric_Pad1.15x1.40mm_HandSolder, F.Cu at (41.9, 106.7)
- added C17: 10n, Capacitor_SMD:C_0805_2012Metric_Pad1.15x1.40mm_HandSolder, F.Cu at (45.7, 99.1)
- added C18: 10n, Capacitor_SMD:C_0805_2012Metric_Pad1.15x1.40mm_HandSolder, F.Cu at (73.7, 60.3)
- added C19: 10n, Capacitor_SMD:C_0805_2012Metric_Pad1.15x1.40mm_HandSolder, F.Cu at (87.8, 45.4)
- added C5: 10n, Capacitor_SMD:C_0805_2012Metric_Pad1.15x1.40mm_HandSolder, F.Cu at (107.2, 53.0)
- added C6: 10n, Capacitor_SMD:C_0805_2012Metric_Pad1.15x1.40mm_HandSolder, F.Cu at (111.9, 53.0)
- added C7: 10n, Capacitor_SMD:C_0805_2012Metric_Pad1.15x1.40mm_HandSolder, F.Cu at (107.2, 55.9)
- added R21: 1k, Resistor_SMD:R_0805_2012Metric_Pad1.15x1.40mm_HandSolder, F.Cu at (36.8, 61.0)
- added R22: 1k, Resistor_SMD:R_0805_2012Metric_Pad1.15x1.40mm_HandSolder, F.Cu at (35.6, 56.5)
- added R23: 820, Resistor_SMD:R_0805_2012Metric_Pad1.15x1.40mm_HandSolder, F.Cu at (46.4, 106.7)
- added R24: 820, Resistor_SMD:R_0805_2012Metric_Pad1.15x1.40mm_HandSolder, F.Cu at (50.8, 106.0)
- added R25: 200, Resistor_SMD:R_0805_2012Metric_Pad1.15x1.40mm_HandSolder, F.Cu at (35.6, 52.1)
- added R26: 200, Resistor_SMD:R_0805_2012Metric_Pad1.15x1.40mm_HandSolder, F.Cu at (40.0, 52.1)
- added R27: 1k, Resistor_SMD:R_0805_2012Metric_Pad1.15x1.40mm_HandSolder, F.Cu at (97.3, 42.4)
- added R28: 820, Resistor_SMD:R_0805_2012Metric_Pad1.15x1.40mm_HandSolder, F.Cu at (88.1, 51.3)
- added R29: 820, Resistor_SMD:R_0805_2012Metric_Pad1.15x1.40mm_HandSolder, F.Cu at (84.4, 54.8)
- added R30: 1k, Resistor_SMD:R_0805_2012Metric_Pad1.15x1.40mm_HandSolder, F.Cu at (92.8, 48.3)
- added R31: 1k, Resistor_SMD:R_0805_2012Metric_Pad1.15x1.40mm_HandSolder, F.Cu at (97.3, 45.4)
- added R32: 1k, Resistor_SMD:R_0805_2012Metric_Pad1.15x1.40mm_HandSolder, F.Cu at (84.4, 57.7)
- added R33: 10k, Resistor_SMD:R_0805_2012Metric_Pad1.15x1.40mm_HandSolder, F.Cu at (45.7, 95.2)
- added RV1: 10k, Potentiometer_THT:Potentiometer_Bourns_3339P_Vertical, F.Cu at (39.4, 97.2)
- added U1: TL072, Package_SO:SOIC-8_3.9x4.9mm_P1.27mm, F.Cu at (43.8, 102.9)
- added U2: TL072, Package_SO:SOIC-8_3.9x4.9mm_P1.27mm, F.Cu at (33.0, 66.0)
- added U3: TL072, Package_SO:SOIC-8_3.9x4.9mm_P1.27mm, F.Cu at (72.0, 53.4)
- moved JP1 117.3 mm to (176.4, 88.4)
- moved C1 117.3 mm to (171.8, 91.1)
- moved J1 117.3 mm to (146.3, 80.1)
- moved J2 117.3 mm to (110.6, 80.1)
- moved J3 117.3 mm to (103.4, 80.1)
- moved R1 117.3 mm to (162.3, 82.2)
- moved R10 117.3 mm to (162.3, 79.3)
- moved R11 117.3 mm to (176.6, 79.3)
- moved R12 117.3 mm to (167.1, 88.1)
- moved R13 117.3 mm to (171.8, 85.2)
- moved R14 117.3 mm to (162.3, 94.0)
- moved R15 117.3 mm to (176.6, 82.2)
- moved R16 117.3 mm to (167.1, 91.1)
- moved R17 117.3 mm to (171.8, 88.1)
- moved R18 117.3 mm to (176.6, 85.2)
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Connections:
- C1 pad 1: Net-(C1-Pad1) -> -12V
Routing:
- net Net-(R1-Pad2): track 27.0 -> 0.00 mm, vias 2 -> 0
- net Net-(R14-Pad2): track 22.8 -> 0.00 mm, vias 2 -> 0
- net Net-(R10-Pad2): track 22.8 -> 0.00 mm, vias 2 -> 0
- net Net-(R12-Pad2): track 22.8 -> 0.00 mm, vias 2 -> 0
- net GND: track 18.7 -> 0.00 mm, vias 2 -> 0
- net Net-(JP1-Pad1): track 18.0 -> 0.00 mm
- net Net-(J1-Pad12): track 12.7 -> 0.00 mm
- net Net-(JP1-Pad2): track 12.5 -> 0.00 mm
- net Net-(J1-Pad6): track 11.0 -> 0.00 mm
- net Net-(J1-Pad8): track 11.0 -> 0.00 mm
- net Net-(J1-Pad10): track 11.0 -> 0.00 mm
- net VCC: track 9.23 -> 0.00 mm
- net Net-(R11-Pad2): track 9.16 -> 0.00 mm
- net Net-(R15-Pad2): track 9.15 -> 0.00 mm
- net Net-(R13-Pad2): track 9.12 -> 0.00 mm
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- removed copper zone on F.Cu, net GND
Other:
- board outline removed
- board text removed: "GND"
- board text removed: "R = 1k"
- board text removed: "R = 2k"
- board text removed: "T"

Commit message: PCB-progress
Parts:
- added C2: 47u, Capacitor_THT:CP_Radial_D6.3mm_P2.50mm, F.Cu at (95.2, 59.7)
- added C20: 47n, Capacitor_SMD:C_0805_2012Metric_Pad1.15x1.40mm_HandSolder, F.Cu at (151.1, 54.6)
- added C21: 47n, Capacitor_SMD:C_0805_2012Metric_Pad1.15x1.40mm_HandSolder, F.Cu at (146.4, 52.5)
- added C22: 100n, Capacitor_SMD:C_0805_2012Metric_Pad1.15x1.40mm_HandSolder, F.Cu at (151.0, 45.8)
- added C23: 100n, Capacitor_SMD:C_0805_2012Metric_Pad1.15x1.40mm_HandSolder, F.Cu at (155.8, 42.8)
- added C24: 15p, Capacitor_SMD:C_0805_2012Metric_Pad1.15x1.40mm_HandSolder, F.Cu at (146.4, 55.5)
- added C25: 10n, Capacitor_SMD:C_0805_2012Metric_Pad1.15x1.40mm_HandSolder, F.Cu at (155.8, 45.8)
- added C26: 10n, Capacitor_SMD:C_0805_2012Metric_Pad1.15x1.40mm_HandSolder, F.Cu at (151.0, 48.7)
- added C27: 100n, Capacitor_SMD:C_0805_2012Metric_Pad1.15x1.40mm_HandSolder, F.Cu at (151.1, 51.7)
- added C28: 100n, Capacitor_SMD:C_0805_2012Metric_Pad1.15x1.40mm_HandSolder, F.Cu at (160.5, 42.8)
- added C29: 100n, Capacitor_SMD:C_0805_2012Metric_Pad1.15x1.40mm_HandSolder, F.Cu at (111.8, 101.6)
- added C3: 47u, Capacitor_THT:CP_Radial_D6.3mm_P2.50mm, F.Cu at (87.6, 59.7)
- added C30: 100n, Capacitor_SMD:C_0805_2012Metric_Pad1.15x1.40mm_HandSolder, F.Cu at (106.7, 111.8)
- added C31: 15p, Capacitor_SMD:C_0805_2012Metric_Pad1.15x1.40mm_HandSolder, F.Cu at (160.5, 45.8)
- added C4: 47u, Capacitor_THT:CP_Radial_D6.3mm_P2.50mm, F.Cu at (82.5, 59.7)
- added FB1: Ferrite_Bead_Small, Resistor_SMD:R_0805_2012Metric_Pad1.15x1.40mm_HandSolder, F.Cu at (97.2, 52.5)
- added FB2: Ferrite_Bead_Small, Resistor_SMD:R_0805_2012Metric_Pad1.15x1.40mm_HandSolder, F.Cu at (89.9, 52.4)
- added FB3: Ferrite_Bead_Small, Resistor_SMD:R_0805_2012Metric_Pad1.15x1.40mm_HandSolder, F.Cu at (82.5, 52.5)
- added J6: Conn_01x03_Male, Connector_PinHeader_2.54mm:PinHeader_1x03_P2.54mm_Vertical, F.Cu at (146.3, 43.7)
- added JP2: Jumper_NO_Small, Resistor_THT:R_Axial_DIN0204_L3.6mm_D1.6mm_P1.90mm_Vertical, F.Cu at (99.6, 53.3)
- added JP3: Jumper_NO_Small, Resistor_THT:R_Axial_DIN0204_L3.6mm_D1.6mm_P1.90mm_Vertical, F.Cu at (92.2, 53.3)
- added JP4: Jumper_NO_Small, Resistor_THT:R_Axial_DIN0204_L3.6mm_D1.6mm_P1.90mm_Vertical, F.Cu at (85.1, 51.6)
- added R34: 4k, Resistor_SMD:R_0805_2012Metric_Pad1.15x1.40mm_HandSolder, F.Cu at (160.5, 48.7)
- added R35: 1k, Resistor_SMD:R_0805_2012Metric_Pad1.15x1.40mm_HandSolder, F.Cu at (155.9, 54.6)
- added R36: 200, Resistor_SMD:R_0805_2012Metric_Pad1.15x1.40mm_HandSolder, F.Cu at (160.6, 51.7)
- added R37: 10k, Resistor_SMD:R_0805_2012Metric_Pad1.15x1.40mm_HandSolder, F.Cu at (160.6, 54.6)
- added U4: LM339, Package_SO:SOIC-14_3.9x8.7mm_P1.27mm, F.Cu at (74.7, 102.1)
- added U5: TL072, Package_SO:SOIC-8_3.9x4.9mm_P1.27mm, F.Cu at (74.7, 91.9)
- J3: value Conn_01x16_Male -> Eurorack Power Connector
- R26: value 200 -> 10k
- moved R26 115.9 mm to (155.9, 51.7)
- moved C13 74.3 mm to (120.4, 112.8), turned to 180 degrees
- moved C14 73.5 mm to (117.3, 109.7), turned to 90 degrees
- moved R27 69.6 mm to (103.6, 111.8), turned to 270 degrees
- moved R32 68.1 mm to (117.3, 117.3), turned to 90 degrees
- moved R28 67.7 mm to (116.3, 112.8), turned to 180 degrees
- moved U2 67.1 mm to (87.9, 104.6)
- moved U3 65.0 mm to (109.2, 106.7)
- moved R31 63.5 mm to (117.3, 105.7), turned to 270 degrees
- moved R29 63.1 mm to (115.3, 109.7), turned to 90 degrees
- moved C18 62.2 mm to (108.7, 111.8), turned to 90 degrees
- moved R30 61.6 mm to (115.3, 105.7), turned to 270 degrees
- moved C19 60.3 mm to (109.7, 101.6), turned to 270 degrees
- moved J5 56.3 mm to (117.3, 133.1), turned to 180 degrees
- moved J2 52.2 mm to (69.6, 47.8), turned to 180 degrees
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Connections:
- J4 pad TN: Net-(J4-PadTN) -> (no net)
- J5 pad TN: Net-(J5-PadTN) -> (no net)
- R26 pad 1: ADC_A_in -> +5V
Routing:
- net +5V: track 0.00 -> 24.7 mm
- net Net-(C14-Pad2): track 0.00 -> 22.5 mm
- net Net-(C12-Pad1): track 0.00 -> 16.3 mm
- net +12V: track 0.00 -> 15.1 mm
- net -12V: track 0.00 -> 13.7 mm
- net Net-(C13-Pad2): track 0.00 -> 12.0 mm
- net GND: track 0.00 -> 10.4 mm
- net Net-(FB3-Pad1): track 0.00 -> 9.56 mm
- net Net-(FB2-Pad1): track 0.00 -> 7.30 mm
- net Net-(FB1-Pad1): track 0.00 -> 6.35 mm
- net Net-(R30-Pad2): track 0.00 -> 6.25 mm
- net Net-(C12-Pad2): track 0.00 -> 5.76 mm
- net Net-(C14-Pad1): track 0.00 -> 4.92 mm
- net Net-(J5-PadT): track 0.00 -> 3.32 mm
Other:
- board outline added: 97.8 x 97.8 mm

Commit message: Schematic
Parts:
- J1: footprint Connector_PinHeader_2.54mm:PinHeader_2x06_P2.54mm_Horizontal -> Connector_PinHeader_2.54mm:PinHeader_2x06_P2.54mm_Vertical
- moved R34 106.1 mm to (65.5, 96.0), turned to 270 degrees
- moved C22 99.3 mm to (68.6, 101.1)
- moved R26 98.9 mm to (68.6, 98.0)
- moved C23 96.2 mm to (80.8, 103.1), turned to 180 degrees
- moved C20 95.8 mm to (68.6, 103.1)
- moved C24 92.3 mm to (65.5, 100.1), turned to 270 degrees
- moved R35 83.7 mm to (81.8, 93.5), turned to 90 degrees
- moved C21 81.6 mm to (80.8, 101.1)
- moved R36 72.9 mm to (90.4, 71.1)
- moved J1 38.7 mm to (113.3, 59.9), turned to 90 degrees
- moved R21 6.86 mm to (61.0, 98.0)
- moved R22 5.59 mm to (61.0, 93.6)
- moved R25 5.58 mm to (61.0, 89.4)
- moved C9 5.23 mm to (57.4, 96.0)
Connections:
- C12 pad 1: Net-(C12-Pad1) -> DAC_R2R_out
- R19 pad 2: DAC_D_out -> DAC_R2R_out
- R28 pad 2: Net-(C12-Pad1) -> DAC_R2R_out
- U3 pad 1: Net-(C12-Pad1) -> DAC_R2R_out
Routing:
- net Net-(C12-Pad1): track 16.3 -> 0.00 mm
- net DAC_R2R_out: track 0.00 -> 16.3 mm
Other:
- board text added: "-12V"
- board text added: "R2R output"

Commit message: PCB
Parts:
- removed C21: 47n, Capacitor_SMD:C_0805_2012Metric_Pad1.15x1.40mm_HandSolder
- removed C23, C27, C28: 100n, Capacitor_SMD:C_0805_2012Metric_Pad1.15x1.40mm_HandSolder
- removed C25, C26: 10n, Capacitor_SMD:C_0805_2012Metric_Pad1.15x1.40mm_HandSolder
- removed R31, R35: 1k, Resistor_SMD:R_0805_2012Metric_Pad1.15x1.40mm_HandSolder
- removed R34: 4k, Resistor_SMD:R_0805_2012Metric_Pad1.15x1.40mm_HandSolder
- removed U5: TL072, Package_SO:SOIC-8_3.9x4.9mm_P1.27mm
- R30: value 1k -> 0; footprint Resistor_SMD:R_0805_2012Metric_Pad1.15x1.40mm_HandSolder -> Resistor_THT:R_Axial_DIN0204_L3.6mm_D1.6mm_P1.90mm_Vertical
- moved J6 77.5 mm to (74.7, 73.2), turned to 180 degrees
- moved R30 44.9 mm to (72.1, 93.5), turned to 180 degrees
Connections:
- C20 pad 2: +12V -> Net-(C20-Pad2)
- C22 pad 2: +12V -> Net-(C20-Pad2)
- R26 pad 1: +5V -> VCC
- R30 pad 1: GND -> Net-(C20-Pad2)
- R30 pad 2: Net-(R30-Pad2) -> +5V
- R36 pad 2: Net-(R35-Pad1) -> (no net)
- U3 pad 6: Net-(R30-Pad2) -> Net-(C14-Pad2)
- U4 pad 10: GND -> Net-(U4-Pad10)
- U4 pad 12: -12V -> GND
- U4 pad 13: GND -> Net-(U4-Pad10)
- U4 pad 14: GND -> Net-(U4-Pad14)
- U4 pad 3: +12V -> Net-(C20-Pad2)
- U4 pad 8: GND -> Net-(U4-Pad14)
Routing:
- net Net-(R30-Pad2): track 6.25 -> 0.00 mm
- net Net-(C14-Pad2): track 22.5 -> 18.7 mm
Other:
- outline, holes or cut-outs redrawn
- board text added: "ADC_A_IN"
- board text added: "ADC_D_OUT"
- board text added: "DAC_D_OUT"
- board text added: "GND +5V"
- board text added: "Input"
- board text added: "Output"
- board text added: "Red Stripe"

Commit message: pcb done?
Parts:
- added D1: BAT43, Diode_THT:D_DO-35_SOD27_P7.62mm_Horizontal, F.Cu at (70.6, 93.0)
- added D2: 3v9, Diode_THT:D_DO-41_SOD81_P10.16mm_Horizontal, F.Cu at (93.0, 87.9)
- added R31: 0, Resistor_THT:R_Axial_DIN0204_L3.6mm_D1.6mm_P1.90mm_Vertical, F.Cu at (67.6, 93.5)
- added R34: 1k, Resistor_SMD:R_0805_2012Metric_Pad1.15x1.40mm_HandSolder, F.Cu at (83.8, 87.9)
- added REF**: MountingHole_3.2mm_M3, MountingHole:MountingHole_3.2mm_M3, F.Cu at (43.7, 134.1)
- added REF**: MountingHole_3.2mm_M3, MountingHole:MountingHole_3.2mm_M3, F.Cu at (131.1, 134.6)
- added REF**: MountingHole_3.2mm_M3, MountingHole:MountingHole_3.2mm_M3, F.Cu at (131.1, 46.7)
- added REF**: MountingHole_3.2mm_M3, MountingHole:MountingHole_3.2mm_M3, F.Cu at (43.2, 46.7)
- moved C31 109.7 mm to (63.5, 97.0), turned to 270 degrees
- moved C1 106.3 mm to (77.2, 122.9), turned to 270 degrees
- moved JP1 102.0 mm to (80.8, 124.0), turned to 90 degrees
- moved R18 96.2 mm to (90.9, 129.0), turned to 270 degrees
- moved R37 95.5 mm to (73.7, 94.0), turned to 270 degrees
- moved R15 91.0 mm to (98.6, 129.0), turned to 270 degrees
- moved R11 89.7 mm to (98.6, 123.4), turned to 270 degrees
- moved R8 88.4 mm to (90.9, 117.9), turned to 270 degrees
- moved R17 88.4 mm to (93.5, 129.0), turned to 270 degrees
- moved R13 87.2 mm to (93.5, 123.4), turned to 270 degrees
- moved R10 86.6 mm to (85.9, 119.9)
- moved R5 82.8 mm to (98.6, 117.9), turned to 270 degrees
- moved R9 82.7 mm to (85.9, 122.4), turned to 180 degrees
- moved C15 82.2 mm to (85.9, 115.8), turned to 180 degrees
- moved R4 81.9 mm to (90.9, 112.3), turned to 270 degrees
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Connections:
- R26 pad 1: VCC -> Net-(R26-Pad1)
- R27 pad 2: DAC_D_out -> Net-(D2-Pad1)
- R36 pad 2: (no net) -> Net-(D1-Pad2)
Routing:
- net +12V: track 15.1 -> 174.3 mm, vias 0 -> 6
- net -12V: track 13.7 -> 153.9 mm, vias 0 -> 2
- net GND: track 10.4 -> 88.5 mm, vias 0 -> 17
- net +5V: track 24.7 -> 87.0 mm, vias 0 -> 1
- net Net-(C31-Pad1): track 0.00 -> 35.6 mm, vias 0 -> 4
- net VCC: track 0.00 -> 31.4 mm
- net Net-(JP1-Pad2): track 0.00 -> 28.7 mm, vias 0 -> 2
- net Net-(R25-Pad2): track 0.00 -> 28.3 mm, vias 0 -> 2
- net Net-(R1-Pad2): track 0.00 -> 25.1 mm, vias 0 -> 2
- net ADC_signal_in: track 0.00 -> 23.9 mm
- net Net-(D2-Pad1): track 0.00 -> 23.7 mm
- net Net-(J1-Pad8): track 0.00 -> 23.5 mm, vias 0 -> 2
- net Net-(J1-Pad7): track 0.00 -> 22.6 mm, vias 0 -> 2
- net Net-(J1-Pad12): track 0.00 -> 22.2 mm
- net Net-(J1-Pad11): track 0.00 -> 21.2 mm
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- added copper zone on B.Cu, net GND

Commit message: HMM
Routing:
- added copper zone on F.Cu, net GND
Other:
- rule trace_min: 0.2 -> 0.127
- board text added: "DSP - Daddy Spiser Peberfrugt"
- board text added: "DTU - Danmarks Tekniske Universitet"
Changed lines of the file:
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@@
   (general
     (thickness 1.6)
-    (drawings 27)
+    (drawings 29)
     (tracks 541)
     (zones 0)
@@
     (0 F.Cu signal)
     (31 B.Cu signal)
-    (32 B.Adhes user)
-    (33 F.Adhes user)
-    (34 B.Paste user)
-    (35 F.Paste user)
+    (32 B.Adhes user hide)
+    (33 F.Adhes user hide)
+    (34 B.Paste user hide)
+    (35 F.Paste user hide)
     (36 B.SilkS user)
     (37 F.SilkS user)
@@
     (zone_clearance 0.508)
     (zone_45_only no)
-    (trace_min 0.2)
+    (trace_min 0.127)
     (via_size 0.8)
     (via_drill 0.4)
@@
       (outputformat 1)
       (mirror false)
-      (drillshape 1)
+      (drillshape 0)
       (scaleselection 1)
-      (outputdirectory ""))
+      (outputdirectory "../"))
   )
   (net 0 "")
@@
     )
   )
+  (gr_text "DTU - Danmarks Tekniske Universitet" (at 105.918 75.311) (layer F.SilkS)
+    (effects (font (size 1 1) (thickness 0.15)) (justify left))
+  )
+  (gr_text "DSP - Daddy Spiser Peberfrugt\n" (at 105.918 73.66) (layer F.SilkS)
+    (effects (font (size 1 1) (thickness 0.15)) (justify left))
+  )
   (gr_text "DAC_D_OUT\n" (at 81.28 85.852) (layer F.SilkS)
     (effects (font (size 1 1) (thickness 0.15)) (justify left))
@@
   (gr_line (start 99.568 59.944) (end 99.568 52.324) (layer F.SilkS) (width 0.12))
   (gr_line (start 77.216 59.944) (end 99.568 59.944) (layer F.SilkS) (width 0.12))
-  (gr_text "Red Stripe\n" (at 103.124 56.896 90) (layer F.SilkS)
+  (gr_text "Red Stripe\n" (at 107.569 56.896 90) (layer F.SilkS)
     (effects (font (size 1 1) (thickness 0.15)))
   )
@@
   (gr_arc (start 134.62 43.18) (end 135.89 43.18) (angle -90) (layer Edge.Cuts) (width 0.05))
   (gr_line (start 77.216 52.832) (end 77.216 59.944) (layer F.SilkS) (width 0.12))
-  (gr_poly (pts (xy 100.584 59.436) (xy 100.076 59.436) (xy 100.076 53.34) (xy 100.584 53.34)) (layer F.SilkS) (width 0.1))
-  (gr_text "-12V\n" (at 101.6 56.896 90) (layer F.SilkS)
+  (gr_poly (pts (xy 105.029 59.436) (xy 104.521 59.436) (xy 104.521 53.34) (xy 105.029 53.34)) (layer F.SilkS) (width 0.1))
+  (gr_text "-12V\n" (at 106.045 56.896 90) (layer F.SilkS)
     (effects (font (size 1 1) (thickness 0.15)))
   )
@@
       )
     )
+  )
+  (zone (net 10) (net_name GND) (layer F.Cu) (hatch edge 0.508)
+    (connect_pads (clearance 0.508))
+    (min_thickness 0.254)
+    (fill yes (arc_segments 32) (thermal_gap 0.508) (thermal_bridge_width 0.508))
+    (polygon
+      (pts
+        (xy 135.128 138.684) (xy 39.116 138.684) (xy 38.608 42.672) (xy 135.128 42.164)
+      )
+    )

Commit message: Arduino tests
Other:
- board text removed: "DSP - Daddy Spiser Peberfrugt"
Changed lines of the file:
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@@
   (general
     (thickness 1.6)
-    (drawings 29)
+    (drawings 28)
     (tracks 541)
     (zones 0)
@@
     (effects (font (size 1 1) (thickness 0.15)) (justify left))
   )
-  (gr_text "DSP - Daddy Spiser Peberfrugt\n" (at 105.918 73.66) (layer F.SilkS)
-    (effects (font (size 1 1) (thickness 0.15)) (justify left))
-  )
